File: hardware/MainBoard.sch (KiCad schematic (older format))
At the start: 65 parts, among them J10 B2_HDR_LEFT, J11 B2_HDR_RIGHT, J9 POWER, Q1 2N3904, Q2 2N3904, Q3 2N3904, U1 ATtiny85, U2 TL074, U3 78L05, U4 79L05

Commit message: [JNTUB-HW] Overhaul PCB layout
- Make traces and clearances much bigger than first attempt
- Remove test points and resistor leading to MCU RESET
- Move some resistors to peripheral board
- Space out remaining components on main board
Parts:
- removed R1, R26, R3, R7, R9: 10k, SDIY:R_Axial_DIN0204_L3.6mm_D1.6mm_P5.08mm_Horizontal, symbol Device:R
- removed TP1: P3_FIN, SDIY:Test_Point, symbol JNTUB-rescue:TEST_1P
- removed TP10: TRG_FIN, SDIY:Test_Point, symbol JNTUB-rescue:TEST_1P
- removed TP12: CLK/TRG, SDIY:Test_Point, symbol JNTUB-rescue:TEST_1P
- removed TP13: OUT, SDIY:Test_Point, symbol JNTUB-rescue:TEST_1P
- removed TP14: PWM_RAW, SDIY:Test_Point, symbol JNTUB-rescue:TEST_1P
- removed TP15: PWM_FILT, SDIY:Test_Point, symbol JNTUB-rescue:TEST_1P
- removed TP2: P2_POT, SDIY:Test_Point, symbol JNTUB-rescue:TEST_1P
- removed TP3: P2_CV, SDIY:Test_Point, symbol JNTUB-rescue:TEST_1P
- removed TP4: P2_FIN, SDIY:Test_Point, symbol JNTUB-rescue:TEST_1P
- removed TP5: P2_SUM, SDIY:Test_Point, symbol JNTUB-rescue:TEST_1P
- removed TP6: P1_POT, SDIY:Test_Point, symbol JNTUB-rescue:TEST_1P
- removed TP7: P1_CV, SDIY:Test_Point, symbol JNTUB-rescue:TEST_1P
- removed TP8: P1_FIN, SDIY:Test_Point, symbol JNTUB-rescue:TEST_1P
- removed TP9: P1_SUM, SDIY:Test_Point, symbol JNTUB-rescue:TEST_1P
- added H2: MountingHole, Mounting_Holes:MountingHole_3.2mm_M3, symbol Mechanical:MountingHole
- C12: value 680p -> C_filt
- R13: value 33k -> 47k
- R18: value 3.3k -> 2.2k
- R20: value 47k -> 100k
- R22: value 47k -> R_filt
- U3: symbol JNTUB-rescue:LM78L05ACZ -> Regulator_Linear:L78L05_TO92
- U4: symbol JNTUB-rescue:LM78L05ACZ -> Regulator_Linear:L79L05_TO92
Connections:
- net P1_CV is gone; now on net CLK_TRG: J11.8 (Pin_8)
- net P1_POT is gone; now on net P2_AVG: J11.9 (Pin_9)
- net P2_CV is gone; now on net MCU_ADC3: J10.8 (Pin_8)
- net P2_POT is gone; now on net P1_AVG: J10.9 (Pin_9)
- net +12V: no longer R19.2
- net +5V: now also J10.1 (Pin_1), R19.2, U1.1 (~RESET~/PB5); no longer J10.2 (Pin_2), J10.5 (Pin_5), J11.5 (Pin_5)
- net -5V: now also J10.2 (Pin_2), U4.2 (VI); no longer J11.2 (Pin_2), U4.1 (OUT)
- net CLK_TRG: no longer J11.7 (Pin_7)
- net GNDREF: now also J10.3 (Pin_3), J10.4 (Pin_4), J10.5 (Pin_5), J11.2 (Pin_2), J11.3 (Pin_3), J11.4 (Pin_4), J11.5 (Pin_5), J11.6 (Pin_6), U4.1 (GND); no longer J10.1 (Pin_1), J10.6 (Pin_6), J11.1 (Pin_1), U4.2 (GND)
- net IN_LED+: now also J11.7 (Pin_7); no longer J11.4 (Pin_4)
- net MCU_ADC3: no longer J10.7 (Pin_7)
- net OUT: now also J11.1 (Pin_1); no longer J11.3 (Pin_3)
- net OUT_LED+: now also J10.7 (Pin_7); no longer J10.4 (Pin_4)
- net OUT_LED-: now also J10.6 (Pin_6); no longer J10.3 (Pin_3)
- net P1_AVG: now reaches U2.5 (+)
- net P2_AVG: now reaches U2.10 (+)
- no-connect marks 1 -> 0
Other:
- note added: "NOTES:\n\n- R_out: Use 1k for 1/4W resistors. Use 2k for 1/8W resistors.\n\n- R_led: Will depend on the color & desired brightness. I use 5.6k for my red LEDs.\n\n- R_filt/C_filt: Set for desired PWM filter freq*.\n For ATtiny85’s max 250kHz PWM, 5kHz cutoff serves well, giving:\n R_filt=47k C_filt=680p\n\n- 10k resistors in PARAM 1 and PARAM 2 can be replaced with anything 10k-100k.\n\n- Schottk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"
- note removed: "(could really be -12V to +12V)"
- note removed: "NOTES:\n\n- R_out: Use 1k for 1/4W resistors.\n Use 2k for 1/8W resistors.\n\n- R_led: Will depend on the color.\n I use XXX for my red LEDs.\n\n- 10k resistors in PARAM 1 and PARAM 2\n can be replaced with anything 10k-100k.\n\n- Schottky diodes in PARAM 1 and PARAM 2\n can be replaced with regular switching diodes,\n but clamping will not be as tight.\n\n- Output is default scaled to -5V/+5V.\n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"
- moved on the sheet: C10, D1, D2, D3, D4, J10, J11, R10, R11, R12, R2, R4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
