File: hardware/JNTUB.kicad_pcb (KiCad board)
At the start: 2 copper layers, 41.1 x 99.1 mm, 76 parts, among them J1 PARAM1_CV, J10 B2_HDR_LEFT, J11 B2_HDR_RIGHT, J12 ISP, J2 PARAM2_CV, J3 CLK/TRG, J4 DITTO, J5 OUT1, J6 OUT2, J7 B1_HDR_LEFT, J8 B1_HDR_RIGHT, J9 POWER, Q1 2N3904, Q2 2N3904, Q3 2N3904, U1 ATtiny85, U2 TL074, U3 78L05, U4 79L05

Commit message: [JNTUB-HW] JNTUB Hardware Revision 0.3
Parts:
- removed the mouse-bite-2.54mm-slot at (216.7, 98.6)
- removed the mouse-bite-2.54mm-slot at (216.7, 153.2)
- removed the mouse-bite-2.54mm-slot at (216.7, 61.5)
- added REF**: Hole_Tooling, SDIY:Hole_Tooling, F.Cu at (235.2, 54.1)
- added REF**: Hole_Tooling, SDIY:Hole_Tooling, F.Cu at (198.1, 54.1)
- added REF**: Hole_Tooling, SDIY:Hole_Tooling, F.Cu at (198.1, 160.8)
- added REF**: Hole_Tooling, SDIY:Hole_Tooling, F.Cu at (235.2, 160.8)
- added mouse-bite-2.54mm-slot: VAL**, Panelization:mouse-bite-2.54mm-slot-long, F.Cu at (216.7, 97.9)
- added mouse-bite-2.54mm-slot: VAL**, Panelization:mouse-bite-2.54mm-slot-long, F.Cu at (216.7, 66.7)
- added mouse-bite-2.54mm-slot: VAL**, Panelization:mouse-bite-2.54mm-slot-long, F.Cu at (216.7, 150.2)
- added mouse-bite-2mm-slot: VAL**, Panelization:mouse-bite-2mm-slot-long-single, F.Cu at (228.1, 57.0)
- added mouse-bite-2mm-slot: VAL**, Panelization:mouse-bite-2mm-slot-long-single, F.Cu at (205.6, 57.0)
- added mouse-bite-2mm-slot: VAL**, Panelization:mouse-bite-2mm-slot-long-single, F.Cu at (227.7, 157.9)
- added mouse-bite-2mm-slot: VAL**, Panelization:mouse-bite-2mm-slot-long-single, F.Cu at (205.2, 157.9)
Other:
- board size 41.1 x 99.1 mm -> 41.1 x 110.7 mm
- board text added: "Feb. 2021"
- board text added: "Rev 0.3"
- board text removed: "Jan. 2021"
- board text removed: "Rev 0.2"
